File: workflow_example.sch (KiCad schematic (older format))
At the start: 4 parts, among them J1 AudioJack2

Commit message: add pcb
Parts:
- J1: footprint (none) -> Connector_Audio:Jack_3.5mm_CUI_SJ-3523-SMT_Horizontal
- R1, R2: footprint (none) -> Resistor_THT:R_Axial_DIN0516_L15.5mm_D5.0mm_P5.08mm_Vertical
- RV1: footprint (none) -> Potentiometer_THT:Potentiometer_Alps_RK09K_Single_Vertical
Changed lines of the file:
@@
 EESchema Schematic File Version 4
+LIBS:workflow_example-cache
 EELAYER 30 0
 EELAYER END
@@
 F 0 "R1" H 4355 2654 50  0000 R CNN
 F 1 "R" H 4355 2745 50  0000 R CNN
-F 2 "" V 4355 2700 50  0001 C CNN
+F 2 "Resistor_THT:R_Axial_DIN0516_L15.5mm_D5.0mm_P5.08mm_Vertical" V 4355 2700 50  0001 C CNN
 F 3 "~" H 4425 2700 50  0001 C CNN
 	1    4425 2700
@@
 F 0 "R2" H 4355 3254 50  0000 R CNN
 F 1 "R" H 4355 3345 50  0000 R CNN
-F 2 "" V 4355 3300 50  0001 C CNN
+F 2 "Resistor_THT:R_Axial_DIN0516_L15.5mm_D5.0mm_P5.08mm_Vertical" V 4355 3300 50  0001 C CNN
 F 3 "~" H 4425 3300 50  0001 C CNN
 	1    4425 3300
@@
 F 0 "RV1" H 4356 3046 50  0000 R CNN
 F 1 "R_POT" H 4356 2955 50  0000 R CNN
-F 2 "" H 4425 3000 50  0001 C CNN
+F 2 "Potentiometer_THT:Potentiometer_Alps_RK09K_Single_Vertical" H 4425 3000 50  0001 C CNN
 F 3 "~" H 4425 3000 50  0001 C CNN
 	1    4425 3000
@@
 F 0 "J1" H 5345 3075 50  0000 R CNN
 F 1 "AudioJack2" H 5345 2984 50  0000 R CNN
-F 2 "" H 5525 3000 50  0001 C CNN
+F 2 "Connector_Audio:Jack_3.5mm_CUI_SJ-3523-SMT_Horizontal" H 5525 3000 50  0001 C CNN
 F 3 "~" H 5525 3000 50  0001 C CNN
 	1    5525 3000
