File: workflow_example.sch (KiCad schematic (older format))
At the start: 4 parts, among them J1 AudioJack2

Commit message: some changes
Parts:
- added R3: R, Resistor_THT:R_Axial_DIN0516_L15.5mm_D5.0mm_P5.08mm_Vertical, symbol Device:R
Connections:
- net at RV1.2: now also R3.2; no longer J1.T
- new net: J1.T, R3.1
Other:
- moved on the sheet: J1
Changed lines of the file:
@@
 L Connector:AudioJack2 J1
 U 1 1 5FA337C3
-P 5850 3000
-F 0 "J1" H 5670 3075 50  0000 R CNN
-F 1 "AudioJack2" H 5670 2984 50  0000 R CNN
-F 2 "Connector_Audio:Jack_3.5mm_CUI_SJ-3523-SMT_Horizontal" H 5850 3000 50  0001 C CNN
-F 3 "~" H 5850 3000 50  0001 C CNN
-	1    5850 3000
+P 5975 2750
+F 0 "J1" H 5795 2825 50  0000 R CNN
+F 1 "AudioJack2" H 5795 2734 50  0000 R CNN
+F 2 "Connector_Audio:Jack_3.5mm_CUI_SJ-3523-SMT_Horizontal" H 5975 2750 50  0001 C CNN
+F 3 "~" H 5975 2750 50  0001 C CNN
+	1    5975 2750
 	-1   0    0    -1
 $EndComp
@@
 L power:GND #PWR01
 U 1 1 5FA34C24
-P 5550 3175
-F 0 "#PWR01" H 5550 2925 50  0001 C CNN
-F 1 "GND" H 5555 3002 50  0000 C CNN
-F 2 "" H 5550 3175 50  0001 C CNN
-F 3 "" H 5550 3175 50  0001 C CNN
-	1    5550 3175
+P 5675 2925
+F 0 "#PWR01" H 5675 2675 50  0001 C CNN
+F 1 "GND" H 5680 2752 50  0000 C CNN
+F 2 "" H 5675 2925 50  0001 C CNN
+F 3 "" H 5675 2925 50  0001 C CNN
+	1    5675 2925
 	1    0    0    -1
 $EndComp
 Wire Wire Line
-	5650 2900 5550 2900
+	5775 2650 5675 2650
 Wire Wire Line
-	5550 2900 5550 3175
+	5675 2650 5675 2925
 Wire Wire Line
 	4425 2400 4425 2550
 Wire Wire Line
 	4425 3450 4425 3675
+$Comp
+L Device:R R3
+U 1 1 5FA39694
+P 5450 2750
+F 0 "R3" H 5380 2704 50  0000 R CNN
+F 1 "R" H 5380 2795 50  0000 R CNN
+F 2 "Resistor_THT:R_Axial_DIN0516_L15.5mm_D5.0mm_P5.08mm_Vertical" V 5380 2750 50  0001 C CNN
+F 3 "~" H 5450 2750 50  0001 C CNN
+	1    5450 2750
+	0    1    1    0
+$EndComp
 Wire Wire Line
-	4575 3000 5650 3000
+	5775 2750 5600 2750
+Wire Wire Line
+	5300 2750 4850 2750
+Wire Wire Line
+	4850 2750 4850 3000
+Wire Wire Line
+	4850 3000 4575 3000
 $EndSCHEMATC
