File: workflow_example.kicad_pcb (KiCad board)
At the start: 2 copper layers, 45 x 30 mm, 4 parts, among them J1 AudioJack2

Commit message: some changes
Parts:
- moved RV1 7.40 mm to (165.2, 75.0)
- moved R2 5.40 mm to (156.2, 70.6), turned to 90 degrees
Routing:
- net Net-(R2-Pad2): track 13.7 -> 10.8 mm
- net Net-(R1-Pad1): track 12.2 -> 14.6 mm
- net Net-(J1-PadT): track 28.1 -> 29.4 mm
Changed lines of the file:
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@@
     (thickness 1.6)
     (drawings 5)
-    (tracks 10)
+    (tracks 12)
     (zones 0)
     (modules 4)
@@
   )
   (module Potentiometer_THT:Potentiometer_Alps_RK09K_Single_Vertical (layer F.Cu)
-    (at 165.2 82.4)
+    (at 165.2 75)
     (descr "Potentiometer, vertical, Alps RK09K Single, http://www.alps.com/prod/info/E/HTML/Potentiometer/RotaryPotentiometers/RK09K/RK09K_list.html")
     (tags "Potentiometer vertical Alps RK09K Single")
@@
   )
   (module Resistor_THT:R_Axial_DIN0516_L15.5mm_D5.0mm_P5.08mm_Vertical (layer F.Cu)
-    (at 156.4 65.2)
+    (at 156.2 70.6 90)
     (descr "Resistor, Axial_DIN0516 series, Axial, Vertical, pin pitch=5.08mm, 2W, length*diameter=15.5*5mm^2, http://cdn-reichelt.de/documents/datenblatt/B400/1_4W%23YAG.pdf")
     (tags "Resistor Axial_DIN0516 series Axial Vertical pin pitch 5.08mm 2W length 15.5mm diameter 5mm")
-    (fp_text reference R2 (at 2.54 -3.62) (layer F.SilkS)
-      (effects (font (size 1 1) (thickness 0.15)))
-    )
-    (fp_text value R (at 2.54 3.62) (layer F.Fab)
-      (effects (font (size 1 1) (thickness 0.15)))
-    )
-    (fp_text user %R (at 2.54 -3.62) (layer F.Fab)
+    (fp_text reference R2 (at 2.54 -3.62 90) (layer F.SilkS)
+      (effects (font (size 1 1) (thickness 0.15)))
+    )
+    (fp_text value R (at 2.54 3.62 90) (layer F.Fab)
+      (effects (font (size 1 1) (thickness 0.15)))
+    )
+    (fp_text user %R (at 2.54 -3.62 90) (layer F.Fab)
       (effects (font (size 1 1) (thickness 0.15)))
     )
@@
     (fp_circle (center 0 0) (end 2.62 0) (layer F.SilkS) (width 0.12))
     (fp_circle (center 0 0) (end 2.5 0) (layer F.Fab) (width 0.1))
-    (pad 2 thru_hole oval (at 5.08 0) (size 2.4 2.4) (drill 1.2) (layers *.Cu *.Mask)
+    (pad 2 thru_hole oval (at 5.08 0 90) (size 2.4 2.4) (drill 1.2) (layers *.Cu *.Mask)
       (net 5 "Net-(R2-Pad2)"))
-    (pad 1 thru_hole circle (at 0 0) (size 2.4 2.4) (drill 1.2) (layers *.Cu *.Mask)
+    (pad 1 thru_hole circle (at 0 0 90) (size 2.4 2.4) (drill 1.2) (layers *.Cu *.Mask)
       (net 2 GND))
     (model ${KISYS3DMOD}/Resistor_THT.3dshapes/R_Axial_DIN0516_L15.5mm_D5.0mm_P5.08mm_Vertical.wrl
@@
   (gr_line (start 180 60) (end 180 90) (layer Edge.Cuts) (width 0.05))
   (gr_line (start 135 60) (end 180 60) (layer Edge.Cuts) (width 0.05))
-  (segment (start 161.9 76.6) (end 165.2 79.9) (width 0.25) (layer F.Cu) (net 1))
-  (segment (start 138.5 76.6) (end 161.9 76.6) (width 0.25) (layer F.Cu) (net 1))
+  (segment (start 138.5 74.95) (end 138.5 76.6) (width 0.25) (layer F.Cu) (net 1))
+  (segment (start 140.95 72.5) (end 138.5 74.95) (width 0.25) (layer F.Cu) (net 1))
+  (segment (start 165.2 72.5) (end 140.95 72.5) (width 0.25) (layer F.Cu) (net 1))
   (segment (start 138.5 65.85) (end 138.5 67.2) (width 0.25) (layer F.Cu) (net 2))
   (segment (start 139.15 65.2) (end 138.5 65.85) (width 0.25) (layer F.Cu) (net 2))
   (segment (start 156.4 65.2) (end 139.15 65.2) (width 0.25) (layer F.Cu) (net 2))
-  (segment (start 164.300001 81.500001) (end 165.2 82.4) (width 0.25) (layer F.Cu) (net 4))
-  (segment (start 156.299999 81.500001) (end 164.300001 81.500001) (width 0.25) (layer F.Cu) (net 4))
   (segment (start 154.2 83.6) (end 156.299999 81.500001) (width 0.25) (layer F.Cu) (net 4))
-  (segment (start 161.48 73.68) (end 165.2 77.4) (width 0.25) (layer F.Cu) (net 5))
-  (segment (start 161.48 65.2) (end 161.48 73.68) (width 0.25) (layer F.Cu) (net 5))
+  (segment (start 158.699999 81.500001) (end 165.2 75) (width 0.25) (layer F.Cu) (net 4))
+  (segment (start 156.299999 81.500001) (end 158.699999 81.500001) (width 0.25) (layer F.Cu) (net 4))
+  (segment (start 156.5864 65.65001) (end 156.2 65.65001) (width 0.25) (layer F.Cu) (net 5))
+  (segment (start 160.85001 65.65001) (end 156.5864 65.65001) (width 0.25) (layer F.Cu) (net 5))
+  (segment (start 165.2 70) (end 160.85001 65.65001) (width 0.25) (layer F.Cu) (net 5))
 )
